Commit message: add upper arm

File: src/robot_description/xacro/robot.xacro (robot description, xacro)
@@ -55,4 +55,41 @@
     </collision>
   </link>
+  <!-- head -->
+  <link name="head0_link">
+    <visual>
+      <geometry>
+        <mesh filename="file://$(find robot_description)/meshes/demo/head_link0.stl"/>
+      </geometry>
+    </visual>
+    <collision>
+      <geometry>
+        <mesh filename="file://$(find robot_description)/meshes/demo/head_link0.stl"/>
+      </geometry>
+    </collision>
+  </link>
+  <link name="head1_link">
+    <visual>
+      <geometry>
+        <mesh filename="file://$(find robot_description)/meshes/demo/head_link1.stl"/>
+      </geometry>
+    </visual>
+    <collision>
+      <geometry>
+        <mesh filename="file://$(find robot_description)/meshes/demo/head_link1.stl"/>
+      </geometry>
+    </collision>
+  </link>
+  <link name="head2_link">
+    <visual>
+      <geometry>
+        <mesh filename="file://$(find robot_description)/meshes/demo/head_link2.stl"/>
+      </geometry>
+    </visual>
+    <collision>
+      <geometry>
+        <mesh filename="file://$(find robot_description)/meshes/demo/head_link2.stl"/>
+      </geometry>
+    </collision>
+  </link>
   <!-- arm -->
   <link name="arm_base_link">
@@ -68,38 +105,51 @@
     </collision>
   </link>
-  <!-- head -->
-  <link name="head0_link">
-    <visual>
-      <geometry>
-        <mesh filename="file://$(find robot_description)/meshes/demo/head_link0.stl"/>
-      </geometry>
-    </visual>
-    <collision>
-      <geometry>
-        <mesh filename="file://$(find robot_description)/meshes/demo/head_link0.stl"/>
-      </geometry>
-    </collision>
-  </link>
-  <link name="head1_link">
-    <visual>
-      <geometry>
-        <mesh filename="file://$(find robot_description)/meshes/demo/head_link1.stl"/>
-      </geometry>
-    </visual>
-    <collision>
-      <geometry>
-        <mesh filename="file://$(find robot_description)/meshes/demo/head_link1.stl"/>
-      </geometry>
-    </collision>
-  </link>
-  <link name="head2_link">
-    <visual>
-      <geometry>
-        <mesh filename="file://$(find robot_description)/meshes/demo/head_link2.stl"/>
-      </geometry>
-    </visual>
-    <collision>
-      <geometry>
-        <mesh filename="file://$(find robot_description)/meshes/demo/head_link2.stl"/>
+  <link name="arm_l0_link">
+    <visual>
+      <geometry>
+        <mesh filename="file://$(find robot_description)/meshes/demo/arm_link0.stl"/>
+      </geometry>
+    </visual>
+    <collision>
+      <geometry>
+        <mesh filename="file://$(find robot_description)/meshes/demo/arm_link0.stl"/>
+      </geometry>
+    </collision>
+  </link>
+  <link name="arm_l1_link">
+    <visual>
+      <geometry>
+        <mesh filename="file://$(find robot_description)/meshes/demo/arm_link1.stl"/>
+      </geometry>
+    </visual>
+    <collision>
+      <geometry>
+        <mesh filename="file://$(find robot_description)/meshes/demo/arm_link1.stl"/>
+      </geometry>
+    </collision>
+  </link>
+  <link name="arm_l2_link">
+    <visual>
+      <geometry>
+        <mesh filename="file://$(find robot_description)/meshes/demo/arm_link2.stl"/>
+      </geometry>
+    </visual>
+    <collision>
+      <geometry>
+        <mesh filename="file://$(find robot_description)/meshes/demo/arm_link2.stl"/>
+      </geometry>
+    </collision>
+  </link>
+  <link name="arm_r0_link">
+    <visual>
+      <origin xyz="0.0 0.0 0.0" rpy="0 0 ${PI}"/>
+      <geometry>
+        <mesh filename="file://$(find robot_description)/meshes/demo/arm_link0.stl"/>
+      </geometry>
+    </visual>
+    <collision>
+      <origin xyz="0.0 0.0 0.0" rpy="0 0 ${PI}"/>
+      <geometry>
+        <mesh filename="file://$(find robot_description)/meshes/demo/arm_link0.stl"/>
       </geometry>
     </collision>
@@ -138,4 +188,26 @@
     <axis xyz="0 0 1"/>
     <limit lower="-${PI_6}" upper="${PI_6}" effort="30" velocity="${PI_4}"/>
+  </joint>
+  <!-- head -->
+  <joint name="head0_joint" type="revolute">
+    <origin xyz="-0.016 0.0 0.073"/>
+    <parent link="arm_base_link"/>
+    <child link="head0_link"/>
+    <axis xyz="0 1 0"/>
+    <limit lower="-${PI_12}" upper="${PI_6}" effort="30" velocity="${PI_4}"/>
+  </joint>
+  <joint name="head1_joint" type="revolute">
+    <origin xyz="0.0 0.0 0.0"/>
+    <parent link="head0_link"/>
+    <child link="head1_link"/>
+    <axis xyz="0 0 1"/>
+    <limit lower="-${PI_2}" upper="${PI_2}" effort="30" velocity="${PI_4}"/>
+  </joint>
+  <joint name="head2_joint" type="revolute">
+    <origin xyz="0.045 0.0 0.165"/>
+    <parent link="head1_link"/>
+    <child link="head2_link"/>
+    <axis xyz="1 0 0"/>
+    <limit lower="-${PI_12}" upper="${PI_12}" effort="30" velocity="${PI_4}"/>
   </joint>
   <!-- arm -->
@@ -146,25 +218,31 @@
     <axis xyz="0 0 0"/>
   </joint>
-  <!-- head -->
-  <joint name="head0_joint" type="revolute">
-    <origin xyz="-0.016 0.0 0.073"/>
+  <joint name="arm_l0_joint" type="revolute">
+    <origin xyz="-0.015335 0.14 0.057294"/>
     <parent link="arm_base_link"/>
-    <child link="head0_link"/>
-    <axis xyz="0 1 0"/>
-    <limit lower="-${PI_12}" upper="${PI_6}" effort="30" velocity="${PI_4}"/>
-  </joint>
-  <joint name="head1_joint" type="revolute">
-    <origin xyz="0.0 0.0 0.0"/>
-    <parent link="head0_link"/>
-    <child link="head1_link"/>
-    <axis xyz="0 0 1"/>
-    <limit lower="-${PI_2}" upper="${PI_2}" effort="30" velocity="${PI_4}"/>
-  </joint>
-  <joint name="head2_joint" type="revolute">
-    <origin xyz="0.045 0.0 0.185"/>
-    <parent link="head1_link"/>
-    <child link="head2_link"/>
+    <child link="arm_l0_link"/>
+    <axis xyz="0 1 0"/>
+    <limit lower="-${PI_2}" upper="${PI_2}" effort="30" velocity="${PI_4}"/>
+  </joint>
+  <joint name="arm_l1_joint" type="revolute">
+    <origin xyz="0.0 0.0 0.0" rpy="${PI_2} 0 0"/>
+    <parent link="arm_l0_link"/>
+    <child link="arm_l1_link"/>
     <axis xyz="1 0 0"/>
-    <limit lower="-${PI_12}" upper="${PI_12}" effort="30" velocity="${PI_4}"/>
+    <limit lower="-${PI_2}" upper="0" effort="30" velocity="${PI_4}"/>
+  </joint>
+  <joint name="arm_l2_joint" type="revolute">
+    <origin xyz="0.0 0.0 -0.1525"/>
+    <parent link="arm_l1_link"/>
+    <child link="arm_l2_link"/>
+    <axis xyz="0 0 1"/>
+    <limit lower="-${PI_2}" upper="${PI_2}" effort="30" velocity="${PI_4}"/>
+  </joint>
+  <joint name="arm_r0_joint" type="revolute">
+    <origin xyz="-0.015335 -0.14 0.057294"/>
+    <parent link="arm_base_link"/>
+    <child link="arm_r0_link"/>
+    <axis xyz="0 1 0"/>
+    <limit lower="-${PI_2}" upper="${PI_2}" effort="30" velocity="${PI_4}"/>
   </joint>
 </robot>

Commit message: add left arm

File: src/robot_description/xacro/robot.xacro (robot description, xacro)
@@ -141,4 +141,41 @@
     </collision>
   </link>
+  <link name="arm_l3_link">
+    <visual>
+      <geometry>
+        <mesh filename="file://$(find robot_description)/meshes/demo/arm_link3.stl"/>
+      </geometry>
+    </visual>
+    <collision>
+      <geometry>
+        <mesh filename="file://$(find robot_description)/meshes/demo/arm_link3.stl"/>
+      </geometry>
+    </collision>
+  </link>
+  <link name="arm_l4_link" />
+  <link name="arm_l5_link">
+    <visual>
+      <geometry>
+        <mesh filename="file://$(find robot_description)/meshes/demo/arm_link4.stl"/>
+      </geometry>
+    </visual>
+    <collision>
+      <geometry>
+        <mesh filename="file://$(find robot_description)/meshes/demo/arm_link4.stl"/>
+      </geometry>
+    </collision>
+  </link>
+  <link name="arm_l6_link">
+    <visual>
+      <geometry>
+        <mesh filename="file://$(find robot_description)/meshes/demo/hand_link0.stl"/>
+      </geometry>
+    </visual>
+    <collision>
+      <geometry>
+        <mesh filename="file://$(find robot_description)/meshes/demo/hand_link0.stl"/>
+      </geometry>
+    </collision>
+  </link>
   <link name="arm_r0_link">
     <visual>
@@ -239,4 +276,32 @@
     <limit lower="-${PI_2}" upper="${PI_2}" effort="30" velocity="${PI_4}"/>
   </joint>
+  <joint name="arm_l3_joint" type="revolute">
+    <origin xyz="0.01 0.0 -0.04"/>
+    <parent link="arm_l2_link"/>
+    <child link="arm_l3_link"/>
+    <axis xyz="0 1 0"/>
+    <limit lower="-${PI_2}" upper="0" effort="30" velocity="${PI_4}"/>
+  </joint>
+  <joint name="arm_l4_joint" type="revolute">
+    <origin xyz="-0.01 0.0 -0.165"/>
+    <parent link="arm_l3_link"/>
+    <child link="arm_l4_link"/>
+    <axis xyz="0 0 1"/>
+    <limit lower="-${PI_2}" upper="${PI_2}" effort="30" velocity="${PI_4}"/>
+  </joint>
+  <joint name="arm_l5_joint" type="revolute">
+    <origin xyz="0.0 0.0 0.0"/>
+    <parent link="arm_l4_link"/>
+    <child link="arm_l5_link"/>
+    <axis xyz="0 1 0"/>
+    <limit lower="-${PI_12}" upper="${PI_12}" effort="30" velocity="${PI_4}"/>
+  </joint>
+  <joint name="arm_l6_joint" type="revolute">
+    <origin xyz="0.0 0.0 -0.05"/>
+    <parent link="arm_l5_link"/>
+    <child link="arm_l6_link"/>
+    <axis xyz="1 0 0"/>
+    <limit lower="-${PI_2}" upper="${PI_2}" effort="30" velocity="${PI_4}"/>
+  </joint>
   <joint name="arm_r0_joint" type="revolute">
     <origin xyz="-0.015335 -0.14 0.057294"/>
